File: cc2564-board.kicad_sch (KiCad schematic)
At the start: 72 parts, among them J1 TYPE-C-31-M-12, J2 Conn_ARM_JTAG_SWD_10, J3 Conn_01x16, J4 Conn_01x16, J5 BOOT, J6 1909763-1, J7 Conn_01x04, SW1 SW_Push, U1 LD1117#33, U2 USBLC6-2P6, U3 LD1117#18, U4 STM32F103C8Tx, U5 TXB0104D, U6 TXB0104D, U7 CC2564CRVMR, Y1 ECS-80-18-30-JGN-TR, Y2 ECS-327MVATX-3-CN-TR, Y3 ECS-260-8-36CKM-TR

Commit message: Swap in TLV711 series 3v3/1v8 dual output LDO
Thanks @noahp for inspiration
Parts:
- removed U1: LD1117#33, Package_TO_SOT_SMD:SOT-223-3_TabPin2, symbol cc2564-board-rescue:AMS1117-3.3-Regulator_Linear
- removed U3: LD1117#18, Package_TO_SOT_SMD:SOT-223-3_TabPin2, symbol cc2564-board-rescue:AMS1117-1.8-Regulator_Linear
- added R18, R19: 10k, Resistor_SMD:R_0402_1005Metric_Pad0.72x0.64mm_HandSolder, symbol cc2564-board-rescue:R-Device
- added U1: TLV7111833DDSET, cc2654-board-footprints:TLV7111833DDSET, symbol LDO-TLV7111833DDSET:TLV7111833DDSET
- C12, C2: value 10uF -> 0.1uF
Connections:
- net GND: now also U1.4 (GND); no longer C12.1
- net VCC_USB: now also R18.2, R19.2, U1.2 (IN); no longer C1.2
- net VDD_1V8: now also C1.2, U1.6 (OUT1); no longer C12.2
- net VDD_3V3: now also U1.5 (OUT2)
- new net: R19.1, U1.1 (EN1)
- new net: R18.1, U1.3 (EN2)
Other:
- note removed: "or ams1117 or rt9193-33"
- moved on the sheet: C10, C3, C4, C5, C6, C7, C8, C9, FB1, J2, L1, R2

Commit message: More board setup pain, route BT fast clock
Parts:
- Y3: footprint cc2654-board-footprints:XTAL_ECS-160-10-36-JGN-TR -> cc2654-board-footprints:XTAL_ECS-260-8-36CKM-TR
Connections:
- net GND: no longer C27.2, U7.B4 (XTALP_FREFP), Y3.1
- net at U7.B5 (MLDO_IN): no longer U7.B6 (CL1-5_LDO_IN)
- new net: C27.2, U7.B4 (XTALP_FREFP), Y3.1
- now unconnected: U7.A2 (DIG_LDO_OUT), U7.A3 (DIG_LDO_OUT), U7.A5 (MLDO_OUT), U7.A9 (MLDO_OUT), U7.B15 (DIG_LDO_OUT), U7.B2 (MLDO_OUT), U7.B26 (DIG_LDO_OUT), U7.B27 (DIG_LDO_OUT), U7.B35 (DIG_LDO_OUT), U7.B36 (DIG_LDO_OUT), U7.B7 (MLDO_OUT)
- no-connect marks 50 -> 63
Changed lines of the file:
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@@
   (junction (at 58.42 91.44) (diameter 1.016) (color 0 0 0 0))
   (junction (at 67.31 327.66) (diameter 1.016) (color 0 0 0 0))
-  (junction (at 73.66 327.66) (diameter 1.016) (color 0 0 0 0))
   (junction (at 73.66 340.36) (diameter 1.016) (color 0 0 0 0))
   (junction (at 74.93 35.56) (diameter 1.016) (color 0 0 0 0))
@@
   (junction (at 180.34 274.32) (diameter 1.016) (color 0 0 0 0))
   (junction (at 180.34 276.86) (diameter 1.016) (color 0 0 0 0))
-  (junction (at 180.34 297.18) (diameter 1.016) (color 0 0 0 0))
-  (junction (at 180.34 299.72) (diameter 1.016) (color 0 0 0 0))
-  (junction (at 180.34 322.58) (diameter 1.016) (color 0 0 0 0))
-  (junction (at 180.34 325.12) (diameter 1.016) (color 0 0 0 0))
-  (junction (at 180.34 327.66) (diameter 1.016) (color 0 0 0 0))
-  (junction (at 180.34 330.2) (diameter 1.016) (color 0 0 0 0))
-  (junction (at 180.34 332.74) (diameter 1.016) (color 0 0 0 0))
   (junction (at 193.04 106.68) (diameter 1.016) (color 0 0 0 0))
   (junction (at 194.31 261.62) (diameter 1.016) (color 0 0 0 0))
@@
   (no_connect (at 255.27 312.42))
   (no_connect (at 39.37 48.26))
+  (no_connect (at 180.34 287.02))
+  (no_connect (at 180.34 289.56))
   (no_connect (at 300.99 279.4))
   (no_connect (at 279.4 142.24))
@@
   (no_connect (at 109.22 279.4))
   (no_connect (at 109.22 284.48))
+  (no_connect (at 180.34 294.64))
+  (no_connect (at 180.34 297.18))
+  (no_connect (at 180.34 299.72))
+  (no_connect (at 180.34 302.26))
   (no_connect (at 255.27 289.56))
+  (no_connect (at 180.34 320.04))
+  (no_connect (at 180.34 322.58))
+  (no_connect (at 180.34 325.12))
+  (no_connect (at 180.34 327.66))
+  (no_connect (at 180.34 330.2))
+  (no_connect (at 180.34 332.74))
+  (no_connect (at 180.34 335.28))
   (no_connect (at 299.72 132.08))
   (no_connect (at 255.27 325.12))
@@
     (stroke (width 0) (type solid) (color 0 0 0 0))
   )
-  (wire (pts (xy 73.66 323.85) (xy 73.66 327.66))
+  (wire (pts (xy 73.66 323.85) (xy 73.66 340.36))
     (stroke (width 0) (type solid) (color 0 0 0 0))
   )
@@
     (stroke (width 0) (type solid) (color 0 0 0 0))
   )
-  (wire (pts (xy 73.66 327.66) (xy 73.66 340.36))
-    (stroke (width 0) (type solid) (color 0 0 0 0))
-  )
   (wire (pts (xy 73.66 340.36) (xy 67.31 340.36))
     (stroke (width 0) (type solid) (color 0 0 0 0))
@@
     (stroke (width 0) (type solid) (color 0 0 0 0))
   )
-  (wire (pts (xy 180.34 287.02) (xy 180.34 289.56))
-    (stroke (width 0) (type solid) (color 0 0 0 0))
-  )
-  (wire (pts (xy 180.34 294.64) (xy 180.34 297.18))
-    (stroke (width 0) (type solid) (color 0 0 0 0))
-  )
-  (wire (pts (xy 180.34 297.18) (xy 180.34 299.72))
-    (stroke (width 0) (type solid) (color 0 0 0 0))
-  )
-  (wire (pts (xy 180.34 299.72) (xy 180.34 302.26))
-    (stroke (width 0) (type solid) (color 0 0 0 0))
-  )
-  (wire (pts (xy 180.34 320.04) (xy 180.34 322.58))
-    (stroke (width 0) (type solid) (color 0 0 0 0))
-  )
-  (wire (pts (xy 180.34 322.58) (xy 180.34 325.12))
-    (stroke (width 0) (type solid) (color 0 0 0 0))
-  )
-  (wire (pts (xy 180.34 325.12) (xy 180.34 327.66))
-    (stroke (width 0) (type solid) (color 0 0 0 0))
-  )
-  (wire (pts (xy 180.34 327.66) (xy 180.34 330.2))
-    (stroke (width 0) (type solid) (color 0 0 0 0))
-  )
-  (wire (pts (xy 180.34 330.2) (xy 180.34 332.74))
-    (stroke (width 0) (type solid) (color 0 0 0 0))
-  )
-  (wire (pts (xy 180.34 332.74) (xy 180.34 335.28))
-    (stroke (width 0) (type solid) (color 0 0 0 0))
-  )
   (wire (pts (xy 182.88 227.33) (xy 180.34 227.33))
     (stroke (width 0) (type solid) (color 0 0 0 0))
@@
       (effects (font (size 1.27 1.27)) (justify left))
     )
-    (property "Footprint" "cc2654-board-footprints:XTAL_ECS-160-10-36-JGN-TR" (id 2) (at 76.2 327.66 0)
+    (property "Footprint" "cc2654-board-footprints:XTAL_ECS-260-8-36CKM-TR" (id 2) (at 76.2 327.66 0)
       (effects (font (size 1.27 1.27)) hide)
     )
@@
     )
     (path "/00000000-0000-0000-0000-00006036c44d"
-      (reference "Y3") (unit 1) (value " ECS-260-8-36CKM-TR") (footprint "cc2654-board-footprints:XTAL_ECS-160-10-36-JGN-TR")
+      (reference "Y3") (unit 1) (value " ECS-260-8-36CKM-TR") (footprint "cc2654-board-footprints:XTAL_ECS-260-8-36CKM-TR")
     )
   )

Commit message: Swap out level shifters for one 8 channel QFN
Parts:
- removed C14, C15, C16, C17: 0.1uF, Capacitor_SMD:C_0402_1005Metric_Pad0.74x0.62mm_HandSolder, symbol cc2564-board-rescue:C-Device
- removed R8, R9: 10k, Resistor_SMD:R_0402_1005Metric_Pad0.72x0.64mm_HandSolder, symbol cc2564-board-rescue:R-Device
- removed U5: TXB0104D, Package_SO:SOIC-14_3.9x8.7mm_P1.27mm, symbol cc2564-board-rescue:TXB0104D-Logic_LevelTranslator
- removed U6: TXB0104D, cc2654-board-footprints:TXB0104D, symbol cc2564-board-rescue:TXB0104D-Logic_LevelTranslator
- added C? (x2): 0.1uF, Capacitor_SMD:C_0402_1005Metric_Pad0.74x0.62mm_HandSolder, symbol cc2564-board-rescue:C-Device
- added R?: 10k, Resistor_SMD:R_0402_1005Metric_Pad0.72x0.64mm_HandSolder, symbol cc2564-board-rescue:R-Device
- added U3: TXB0108DQSR, cc2654-board-footprints:TXB0108DQSR, symbol TXB0108DQSR:TXB0108DQSR
Connections:
- net GND: now also C?.1, C?.1, U3.15 (GND)
- net NSHUTDOWN: now also U3.7 (A5)
- net NSHUTDOWN_1V8: now also U3.14 (B5)
- net USART2_CTS: now also U3.1 (A1)
- net USART2_CTS_1V8: now also U3.20 (B1)
- net USART2_RTS: now also U3.2 (A2)
- net USART2_RTS_1V8: now also U3.19 (B2)
- net USART2_RX: now also U3.4 (A4)
- net USART2_RX_1V8: now also U3.17 (B4)
- net USART2_TX: now also U3.3 (A3)
- net USART2_TX_1V8: now also U3.18 (B3)
- net VDD_1V8: now also C?.2, U3.16 (VCCB)
- net VDD_3V3: now also C?.2, R?.1, U3.5 (VCCA)
- new net: R?.2, U3.6 (OE)
Other:
- moved on the sheet: D1, D2, D3, J3, J4, R5, R6, R7

Commit message: Begin serious layout
Parts:
- gave numbers to parts that had none: 3
- renumbered C3 to C1, C2 to C10, C18 to C16, C19 to C17, C20 to C18, C21 to C19, C4 to C2, C22 to C20, C23 to C21, C24 to C22, C25 to C23, C26 to C24, C27 to C25, C28 to C26, C5 to C3, C6 to C4, C7 to C5, C1 to C6, C8 to C7, C9 to C8, C10 to C9, R2 to R1, R7 to R10, R10 to R11, R11 to R12, R12 to R13, R13 to R14, R14 to R15, R15 to R16, R16 to R17, R17 to R18, R1 to R2, R18 to R3, R19 to R4, R3 to R5, R4 to R6, R5 to R8, R6 to R9, U4 to U3, U3 to U4, U7 to U5
Connections:
- net USB_CONN_D+: now also U2.6 (I/O1); no longer U2.4 (I/O2)
- net USB_CONN_D-: now also U2.4 (I/O2); no longer U2.6 (I/O1)
- net USB_D+: now also U2.1 (I/O1); no longer U2.3 (I/O2)
- net USB_D-: now also U2.3 (I/O2); no longer U2.1 (I/O1)

Commit message: Finish most BT stuff
Parts:
- removed C12: 0.1uF, Capacitor_SMD:C_0402_1005Metric_Pad0.74x0.62mm_HandSolder, symbol cc2564-board-rescue:C-Device
Connections:
- net GND: now also C25.2, U5.B4 (XTALP_FREFP), Y3.1
Changed lines of the file:
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@@
   (junction (at 58.42 91.44) (diameter 1.016) (color 0 0 0 0))
   (junction (at 67.31 327.66) (diameter 1.016) (color 0 0 0 0))
+  (junction (at 73.66 327.66) (diameter 1.016) (color 0 0 0 0))
   (junction (at 73.66 340.36) (diameter 1.016) (color 0 0 0 0))
   (junction (at 74.93 35.56) (diameter 1.016) (color 0 0 0 0))
@@
   (junction (at 431.8 48.26) (diameter 1.016) (color 0 0 0 0))
   (junction (at 477.52 48.26) (diameter 1.016) (color 0 0 0 0))
-  (no_connect (at 255.27 299.72))
-  (no_connect (at 109.22 287.02))
-  (no_connect (at 255.27 294.64))
-  (no_connect (at 300.99 304.8))
+  (no_connect (at 180.34 330.2))
+  (no_connect (at 255.27 304.8))
+  (no_connect (at 302.26 55.88))
   (no_connect (at 255.27 279.4))
-  (no_connect (at 300.99 297.18))
-  (no_connect (at 88.9 120.65))
-  (no_connect (at 180.34 314.96))
-  (no_connect (at 300.99 307.34))
-  (no_connect (at 180.34 309.88))
+  (no_connect (at 109.22 281.94))
+  (no_connect (at 255.27 317.5))
+  (no_connect (at 255.27 312.42))
   (no_connect (at 300.99 292.1))
-  (no_connect (at 255.27 292.1))
-  (no_connect (at 255.27 320.04))
+  (no_connect (at 180.34 314.96))
+  (no_connect (at 251.46 148.59))
+  (no_connect (at 255.27 297.18))
+  (no_connect (at 180.34 327.66))
   (no_connect (at 180.34 312.42))
-  (no_connect (at 300.99 302.26))
-  (no_connect (at 300.99 287.02))
-  (no_connect (at 300.99 284.48))
+  (no_connect (at 109.22 279.4))
   (no_connect (at 109.22 314.96))
-  (no_connect (at 255.27 314.96))
-  (no_connect (at 300.99 299.72))
-  (no_connect (at 255.27 317.5))
-  (no_connect (at 255.27 297.18))
   (no_connect (at 88.9 123.19))
-  (no_connect (at 300.99 281.94))
-  (no_connect (at 74.93 43.18))
-  (no_connect (at 255.27 304.8))
-  (no_connect (at 300.99 289.56))
-  (no_connect (at 255.27 312.42))
-  (no_connect (at 39.37 48.26))
-  (no_connect (at 180.34 287.02))
+  (no_connect (at 300.99 302.26))
+  (no_connect (at 180.34 320.04))
+  (no_connect (at 180.34 302.26))
   (no_connect (at 180.34 289.56))
-  (no_connect (at 300.99 279.4))
-  (no_connect (at 109.22 281.94))
-  (no_connect (at 255.27 302.26))
+  (no_connect (at 180.34 322.58))
   (no_connect (at 255.27 307.34))
-  (no_connect (at 255.27 287.02))
-  (no_connect (at 251.46 130.81))
+  (no_connect (at 180.34 309.88))
+  (no_connect (at 300.99 281.94))
+  (no_connect (at 300.99 299.72))
+  (no_connect (at 109.22 287.02))
+  (no_connect (at 251.46 143.51))
   (no_connect (at 251.46 133.35))
+  (no_connect (at 255.27 322.58))
+  (no_connect (at 255.27 292.1))
+  (no_connect (at 255.27 294.64))
+  (no_connect (at 180.34 297.18))
   (no_connect (at 251.46 135.89))
-  (no_connect (at 251.46 143.51))
-  (no_connect (at 251.46 146.05))
-  (no_connect (at 251.46 148.59))
+  (no_connect (at 39.37 48.26))
+  (no_connect (at 255.27 287.02))
   (no_connect (at 88.9 118.11))
-  (no_connect (at 255.27 322.58))
-  (no_connect (at 302.26 55.88))
+  (no_connect (at 180.34 325.12))
+  (no_connect (at 180.34 332.74))
+  (no_connect (at 88.9 120.65))
+  (no_connect (at 255.27 299.72))
+  (no_connect (at 255.27 325.12))
   (no_connect (at 180.34 307.34))
-  (no_connect (at 109.22 279.4))
-  (no_connect (at 109.22 284.48))
+  (no_connect (at 300.99 287.02))
   (no_connect (at 180.34 294.64))
-  (no_connect (at 180.34 297.18))
+  (no_connect (at 300.99 279.4))
+  (no_connect (at 255.27 314.96))
   (no_connect (at 180.34 299.72))
-  (no_connect (at 180.34 302.26))
+  (no_connect (at 74.93 43.18))
+  (no_connect (at 251.46 130.81))
+  (no_connect (at 300.99 294.64))
+  (no_connect (at 300.99 284.48))
+  (no_connect (at 255.27 309.88))
+  (no_connect (at 300.99 297.18))
   (no_connect (at 255.27 289.56))
-  (no_connect (at 180.34 320.04))
-  (no_connect (at 180.34 322.58))
-  (no_connect (at 180.34 325.12))
-  (no_connect (at 180.34 327.66))
-  (no_connect (at 180.34 330.2))
-  (no_connect (at 180.34 332.74))
+  (no_connect (at 300.99 289.56))
+  (no_connect (at 180.34 287.02))
+  (no_connect (at 251.46 146.05))
+  (no_connect (at 300.99 304.8))
+  (no_connect (at 109.22 284.48))
+  (no_connect (at 255.27 302.26))
   (no_connect (at 180.34 335.28))
-  (no_connect (at 255.27 325.12))
-  (no_connect (at 255.27 309.88))
-  (no_connect (at 300.99 294.64))
+  (no_connect (at 300.99 307.34))
+  (no_connect (at 255.27 320.04))
   (wire (pts (xy 21.59 40.64) (xy 39.37 40.64))
     (stroke (width 0) (type solid) (color 0 0 0 0))
@@
     (stroke (width 0) (type solid) (color 0 0 0 0))
   )
-  (wire (pts (xy 73.66 323.85) (xy 73.66 340.36))
+  (wire (pts (xy 73.66 323.85) (xy 73.66 327.66))
     (stroke (width 0) (type solid) (color 0 0 0 0))
   )
@@
     (stroke (width 0) (type solid) (color 0 0 0 0))
   )
+  (wire (pts (xy 73.66 327.66) (xy 73.66 340.36))
+    (stroke (width 0) (type solid) (color 0 0 0 0))
+  )
   (wire (pts (xy 73.66 340.36) (xy 67.31 340.36))
     (stroke (width 0) (type solid) (color 0 0 0 0))
@@
     )
   )
-  (symbol (lib_id "cc2564-board-rescue:C-Device") (at 124.46 93.98 180) (unit 1)
-    (in_bom yes) (on_board yes)
-    (property "Reference" "C12" (id 0) (at 121.539 95.1484 0)
-      (effects (font (size 1.27 1.27)) (justify left))
-    )
-    (property "Value" "0.1uF" (id 1) (at 121.539 92.837 0)
-      (effects (font (size 1.27 1.27)) (justify left))
-    )
-    (property "Footprint" "Capacitor_SMD:C_0402_1005Metric_Pad0.74x0.62mm_HandSolder" (id 2) (at 123.4948 90.17 0)
-      (effects (font (size 1.27 1.27)) hide)
-    )
-    (property "Datasheet" "~" (id 3) (at 124.46 93.98 0)
-      (effects (font (size 1.27 1.27)) hide)
-    )
-  )
   (symbol (lib_id "cc2564-board-rescue:C-Device") (at 166.37 59.69 180) (unit 1)
     (in_bom yes) (on_board yes)
@@
       (reference "C11") (unit 1) (value "0.1uF") (footprint "Capacitor_SMD:C_0402_1005Metric_Pad0.74x0.62mm_HandSolder")
     )
-    (path "/64accb6f-f295-4d56-a3e5-87b6fb02ba69"
-      (reference "C12") (unit 1) (value "0.1uF") (footprint "Capacitor_SMD:C_0402_1005Metric_Pad0.74x0.62mm_HandSolder")
-    )
     (path "/00000000-0000-0000-0000-00005fe651dc"
